File: homeWork2.kicad_sch (KiCad schematic)
At the start: 53 parts, among them J1 Barrel_Jack_Switch_SMT, J2 Conn_01x15_Socket, J3 Conn_01x15_Socket, J4_LCD1 Conn_01x04_Socket_LCD, J5_DFPLAYER1 Conn_01x04_Socket_DFPLAYER, U1 LM7805_TO220

Commit message: Adding additional JLCPCB partnumbers.
Parts:
- J2, J3: Cost (none) -> 0.0989; Distributor 1 (none) -> JLCPCB; Distributor 1 PN (none) -> C7509525
- J4_LCD1, J5_DFPLAYER1: Cost (none) -> 0.0378; Distributor 1 (none) -> JLCPCB; Distributor 1 PN (none) -> C7509546
Changed lines of the file:
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@@
+      (effects (font (size 1.27 1.27)) hide)
+    )
+    (property "Description" "2.54mm Plugin Gold Straight 1x15P 8.5mm Plugin,P=2.54mm Female Headers ROHS" (at 130.81 99.06 0)
+      (effects (font (size 1.27 1.27)) hide)
+    )
+    (property "Distributor 1" "JLCPCB" (at 130.81 99.06 0)
+      (effects (font (size 1.27 1.27)) hide)
+    )
+    (property "Distributor 1 PN" "C7509525" (at 130.81 99.06 0)
+      (effects (font (size 1.27 1.27)) hide)
+    )
+    (property "Cost" "0.0989" (at 130.81 99.06 0)
       (effects (font (size 1.27 1.27)) hide)
     )
@@
       (effects (font (size 1.27 1.27)) hide)
     )
+    (property "Description" "2.54mm Plugin Gold Straight 1x4P 8.5mm Plugin,P=2.54mm Female Headers ROHS" (at 171.45 57.15 0)
+      (effects (font (size 1.27 1.27)) hide)
+    )
+    (property "Distributor 1" "JLCPCB" (at 171.45 57.15 0)
+      (effects (font (size 1.27 1.27)) hide)
+    )
+    (property "Distributor 1 PN" "C7509546" (at 171.45 57.15 0)
+      (effects (font (size 1.27 1.27)) hide)
+    )
+    (property "Cost" "0.0378" (at 171.45 57.15 0)
+      (effects (font (size 1.27 1.27)) hide)
+    )
     (pin "1")
     (pin "2")
@@
       (effects (font (size 1.27 1.27)) hide)
     )
+    (property "Description" "2.54mm Plugin Gold Straight 1x4P 8.5mm Plugin,P=2.54mm Female Headers ROHS" (at 140.97 67.31 0)
+      (effects (font (size 1.27 1.27)) hide)
+    )
+    (property "Distributor 1" "JLCPCB" (at 140.97 67.31 0)
+      (effects (font (size 1.27 1.27)) hide)
+    )
+    (property "Distributor 1 PN" "C7509546" (at 140.97 67.31 0)
+      (effects (font (size 1.27 1.27)) hide)
+    )
+    (property "Cost" "0.0378" (at 140.97 67.31 0)
+      (effects (font (size 1.27 1.27)) hide)
+    )
     (pin "1")
     (pin "2")
@@
       (effects (font (size 1.27 1.27)) hide)
     )
+    (property "Description" "2.54mm Plugin Gold Straight 1x15P 8.5mm Plugin,P=2.54mm Female Headers ROHS" (at 93.98 99.06 0)
+      (effects (font (size 1.27 1.27)) hide)
+    )
+    (property "Distributor 1" "JLCPCB" (at 93.98 99.06 0)
+      (effects (font (size 1.27 1.27)) hide)
+    )
+    (property "Distributor 1 PN" "C7509525" (at 93.98 99.06 0)
+      (effects (font (size 1.27 1.27)) hide)
+    )
+    (property "Cost" "0.0989" (at 93.98 99.06 0)
+      (effects (font (size 1.27 1.27)) hide)
+    )
