File: homeWork2.kicad_sch (KiCad schematic)
At the start: 53 parts, among them J1 Barrel_Jack_Switch_SMT, J2 Conn_01x15_Socket, J3 Conn_01x15_Socket, J4_LCD1 Conn_01x04_Socket_LCD, J5_DFPLAYER1 Conn_01x04_Socket_DFPLAYER, U1 LM7805_TO220

Commit message: Updated the parts for available parts manufacturing.
Parts:
- D2: Cost 0.0343 -> 0.0228
- ESP32_DEVKITV1: value ~ -> ESP32-DEVKIT1
- J4_LCD1: value Conn_01x04_Socket_LCD -> Conn_01x04
- J5_DFPLAYER1: value Conn_01x04_Socket_DFPLAYER -> Conn_01x04
- R1: value 1R -> 1
- R10, R11, R12, R13, R14, R8, R9: value 60 ohm -> 62; Cost 0.0015 -> 0.0017; Distributor 1 PN C269711 -> C269429
- R2: value 330R -> 150; Distributor 1 PN C269711 -> C325599
- R3, R4, R5, R6: value 10 k -> 10k
- R7: value 1R -> 1; Cost 0.0015 -> 0.0020
- TP1, TP2, TP3, TP4, TP5: Cost (none) -> 0.0696; Distributor 1 (none) -> JLCPCB; Distributor 1 PN (none) -> C5277086
Other:
- note added: "Red LED Forward current (I) = 20 mA = 0.02 A Voltage across Red LED (V_LED) = 2.04 V ESP32 GPIO output voltage (V_GPIO) = 5 V To calculate the resistor value (R): R= (V GPIO - V LED) / I R= (5 V - 2.04 V) / 0.02 A R= 2.96 v / 0.02 A R= 148 Ω"

Commit message: Added firmware.
Parts:
- J1: Manufacturier XKB Connectivity / Tensility International Corp -> (none)
- J2, J3: MPN (none) -> DS1023-1x15SF11; Manufacturer (none) -> CONNFLY Elec
- J4_LCD1, J5_DFPLAYER1: MPN (none) -> DS1023-1x4SF11; Manufacturer (none) -> CONNFLY Elec
- S1-morseCodeDanger1, S2-RepeatCalculation1, S3-muteFiveMin1, S4-SendEmergMessage1: M2PN (none) -> C13828; Manufacturer 2 (none) -> Dongguan Guangzhu Industrial
- TP1, TP2, TP3, TP4, TP5: MPN (none) -> RH-5000; Manufacturer (none) -> ronghe
