File: homeWork2/homeWork2.kicad_sch (KiCad schematic)
At the start: 53 parts, among them J1 Barrel_Jack_Switch_SMT, J2 Conn_01x15_Socket, J3 Conn_01x15_Socket, J4_LCD1 Conn_01x04, J5_DFPLAYER1 Conn_01x04, U1 LM7805_TO220

Commit message: Updated the switches and added 3d model for the switches.
Parts:
- S1-morseCodeDanger1, S2-RepeatCalculation1, S3-muteFiveMin1, S4-SendEmergMessage1: footprint GeneralPurposeAlarmDevicePCB:Switch_Tactile_THT_6x6mm -> Button_Switch_THT:SW_PUSH_6mm_H9.5mm
Changed lines of the file:
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@@
       (effects (font (size 1.524 1.524)))
     )
-    (property "Footprint" "GeneralPurposeAlarmDevicePCB:Switch_Tactile_THT_6x6mm" (at 67.31 69.85 0)
+    (property "Footprint" "Button_Switch_THT:SW_PUSH_6mm_H9.5mm" (at 67.31 69.85 0)
       (effects (font (size 1.524 1.524)) (justify left) hide)
     )
@@
       (effects (font (size 1.524 1.524)))
     )
-    (property "Footprint" "GeneralPurposeAlarmDevicePCB:Switch_Tactile_THT_6x6mm" (at 67.31 87.63 0)
+    (property "Footprint" "Button_Switch_THT:SW_PUSH_6mm_H9.5mm" (at 67.31 87.63 0)
       (effects (font (size 1.524 1.524)) (justify left) hide)
     )
@@
       (effects (font (size 1.524 1.524)))
     )
-    (property "Footprint" "GeneralPurposeAlarmDevicePCB:Switch_Tactile_THT_6x6mm" (at 67.31 102.87 0)
+    (property "Footprint" "Button_Switch_THT:SW_PUSH_6mm_H9.5mm" (at 67.31 102.87 0)
       (effects (font (size 1.524 1.524)) (justify left) hide)
     )
@@
       (effects (font (size 1.524 1.524)))
     )
-    (property "Footprint" "GeneralPurposeAlarmDevicePCB:Switch_Tactile_THT_6x6mm" (at 67.31 52.07 0)
-      (effects (font (size 1.524 1.524)) (justify left) hide)
-    )
+    (property "Footprint" "Button_Switch_THT:SW_PUSH_6mm_H9.5mm" (at 67.31 52.07 0)
+      (effects (font (size 1.524 1.524)) (justify left) hide)
+    )
